Commit message: created a new folder for planner examples, started converting basic_cartesian_example from trajopt example to planner example

File: tesseract_ros/tesseract_examples/tesseract_examples_support/urdf/car_seat_demo_macro.xacro (robot description, xacro)
@@ -7,5 +7,5 @@
             <origin rpy="0 0 0" xyz="0 0 0"/>
             <geometry>
-              <mesh filename="package://trajopt_ros_examples/meshes/car_seat/visual/car.stl"/>
+              <mesh filename="package://tesseract_ros_examples/meshes/car_seat/visual/car.stl"/>
             </geometry>
             <material name="gray">
@@ -15,120 +15,120 @@
           <collision>
             <geometry>
-              <mesh filename="package://trajopt_ros_examples/meshes/car_seat/collision/car_1.stl"/>
-            </geometry>
-          </collision>
-          <collision>
-            <geometry>
-              <mesh filename="package://trajopt_ros_examples/meshes/car_seat/collision/car_2.stl"/>
-            </geometry>
-          </collision>
-          <collision>
-            <geometry>
-              <mesh filename="package://trajopt_ros_examples/meshes/car_seat/collision/car_3.stl"/>
-            </geometry>
-          </collision>
-          <collision>
-            <geometry>
-              <mesh filename="package://trajopt_ros_examples/meshes/car_seat/collision/car_4.stl"/>
-            </geometry>
-          </collision>
-          <collision>
-            <geometry>
-              <mesh filename="package://trajopt_ros_examples/meshes/car_seat/collision/car_5.stl"/>
-            </geometry>
-          </collision>
-          <collision>
-            <geometry>
-              <mesh filename="package://trajopt_ros_examples/meshes/car_seat/collision/car_6.stl"/>
-            </geometry>
-          </collision>
-          <collision>
-            <geometry>
-              <mesh filename="package://trajopt_ros_examples/meshes/car_seat/collision/car_7.stl"/>
-            </geometry>
-          </collision>
-          <collision>
-            <geometry>
-              <mesh filename="package://trajopt_ros_examples/meshes/car_seat/collision/car_8.stl"/>
-            </geometry>
-          </collision>
-          <collision>
-            <geometry>
-              <mesh filename="package://trajopt_ros_examples/meshes/car_seat/collision/car_9.stl"/>
-            </geometry>
-          </collision>
-          <collision>
-            <geometry>
-              <mesh filename="package://trajopt_ros_examples/meshes/car_seat/collision/car_10.stl"/>
-            </geometry>
-          </collision>
-          <collision>
-            <geometry>
-              <mesh filename="package://trajopt_ros_examples/meshes/car_seat/collision/car_11.stl"/>
-            </geometry>
-          </collision>
-          <collision>
-            <geometry>
-              <mesh filename="package://trajopt_ros_examples/meshes/car_seat/collision/car_12.stl"/>
-            </geometry>
-          </collision>
-          <collision>
-            <geometry>
-              <mesh filename="package://trajopt_ros_examples/meshes/car_seat/collision/car_13.stl"/>
-            </geometry>
-          </collision>
-          <collision>
-            <geometry>
-              <mesh filename="package://trajopt_ros_examples/meshes/car_seat/collision/car_14.stl"/>
-            </geometry>
-          </collision>
-          <collision>
-            <geometry>
-              <mesh filename="package://trajopt_ros_examples/meshes/car_seat/collision/car_15.stl"/>
-            </geometry>
-          </collision>
-          <collision>
-            <geometry>
-              <mesh filename="package://trajopt_ros_examples/meshes/car_seat/collision/car_16.stl"/>
-            </geometry>
-          </collision>
-          <collision>
-            <geometry>
-              <mesh filename="package://trajopt_ros_examples/meshes/car_seat/collision/car_17.stl"/>
-            </geometry>
-          </collision>
-          <collision>
-            <geometry>
-              <mesh filename="package://trajopt_ros_examples/meshes/car_seat/collision/car_18.stl"/>
-            </geometry>
-          </collision>
-          <collision>
-            <geometry>
-              <mesh filename="package://trajopt_ros_examples/meshes/car_seat/collision/car_19.stl"/>
-            </geometry>
-          </collision>
-          <collision>
-            <geometry>
-              <mesh filename="package://trajopt_ros_examples/meshes/car_seat/collision/car_20.stl"/>
-            </geometry>
-          </collision>
-          <collision>
-            <geometry>
-              <mesh filename="package://trajopt_ros_examples/meshes/car_seat/collision/car_21.stl"/>
-            </geometry>
-          </collision>
-          <collision>
-            <geometry>
-              <mesh filename="package://trajopt_ros_examples/meshes/car_seat/collision/car_22.stl"/>
-            </geometry>
-          </collision>
-          <collision>
-            <geometry>
-              <mesh filename="package://trajopt_ros_examples/meshes/car_seat/collision/car_23.stl"/>
-            </geometry>
-          </collision>
-          <collision>
-            <geometry>
-              <mesh filename="package://trajopt_ros_examples/meshes/car_seat/collision/car_24.stl"/>
+              <mesh filename="package://tesseract_ros_examples/meshes/car_seat/collision/car_1.stl"/>
+            </geometry>
+          </collision>
+          <collision>
+            <geometry>
+              <mesh filename="package://tesseract_ros_examples/meshes/car_seat/collision/car_2.stl"/>
+            </geometry>
+          </collision>
+          <collision>
+            <geometry>
+              <mesh filename="package://tesseract_ros_examples/meshes/car_seat/collision/car_3.stl"/>
+            </geometry>
+          </collision>
+          <collision>
+            <geometry>
+              <mesh filename="package://tesseract_ros_examples/meshes/car_seat/collision/car_4.stl"/>
+            </geometry>
+          </collision>
+          <collision>
+            <geometry>
+              <mesh filename="package://tesseract_ros_examples/meshes/car_seat/collision/car_5.stl"/>
+            </geometry>
+          </collision>
+          <collision>
+            <geometry>
+              <mesh filename="package://tesseract_ros_examples/meshes/car_seat/collision/car_6.stl"/>
+            </geometry>
+          </collision>
+          <collision>
+            <geometry>
+              <mesh filename="package://tesseract_ros_examples/meshes/car_seat/collision/car_7.stl"/>
+            </geometry>
+          </collision>
+          <collision>
+            <geometry>
+              <mesh filename="package://tesseract_ros_examples/meshes/car_seat/collision/car_8.stl"/>
+            </geometry>
+          </collision>
+          <collision>
+            <geometry>
+              <mesh filename="package://tesseract_ros_examples/meshes/car_seat/collision/car_9.stl"/>
+            </geometry>
+          </collision>
+          <collision>
+            <geometry>
+              <mesh filename="package://tesseract_ros_examples/meshes/car_seat/collision/car_10.stl"/>
+            </geometry>
+          </collision>
+          <collision>
+            <geometry>
+              <mesh filename="package://tesseract_ros_examples/meshes/car_seat/collision/car_11.stl"/>
+            </geometry>
+          </collision>
+          <collision>
+            <geometry>
+              <mesh filename="package://tesseract_ros_examples/meshes/car_seat/collision/car_12.stl"/>
+            </geometry>
+          </collision>
+          <collision>
+            <geometry>
+              <mesh filename="package://tesseract_ros_examples/meshes/car_seat/collision/car_13.stl"/>
+            </geometry>
+          </collision>
+          <collision>
+            <geometry>
+              <mesh filename="package://tesseract_ros_examples/meshes/car_seat/collision/car_14.stl"/>
+            </geometry>
+          </collision>
+          <collision>
+            <geometry>
+              <mesh filename="package://tesseract_ros_examples/meshes/car_seat/collision/car_15.stl"/>
+            </geometry>
+          </collision>
+          <collision>
+            <geometry>
+              <mesh filename="package://tesseract_ros_examples/meshes/car_seat/collision/car_16.stl"/>
+            </geometry>
+          </collision>
+          <collision>
+            <geometry>
+              <mesh filename="package://tesseract_ros_examples/meshes/car_seat/collision/car_17.stl"/>
+            </geometry>
+          </collision>
+          <collision>
+            <geometry>
+              <mesh filename="package://tesseract_ros_examples/meshes/car_seat/collision/car_18.stl"/>
+            </geometry>
+          </collision>
+          <collision>
+            <geometry>
+              <mesh filename="package://tesseract_ros_examples/meshes/car_seat/collision/car_19.stl"/>
+            </geometry>
+          </collision>
+          <collision>
+            <geometry>
+              <mesh filename="package://tesseract_ros_examples/meshes/car_seat/collision/car_20.stl"/>
+            </geometry>
+          </collision>
+          <collision>
+            <geometry>
+              <mesh filename="package://tesseract_ros_examples/meshes/car_seat/collision/car_21.stl"/>
+            </geometry>
+          </collision>
+          <collision>
+            <geometry>
+              <mesh filename="package://tesseract_ros_examples/meshes/car_seat/collision/car_22.stl"/>
+            </geometry>
+          </collision>
+          <collision>
+            <geometry>
+              <mesh filename="package://tesseract_ros_examples/meshes/car_seat/collision/car_23.stl"/>
+            </geometry>
+          </collision>
+          <collision>
+            <geometry>
+              <mesh filename="package://tesseract_ros_examples/meshes/car_seat/collision/car_24.stl"/>
             </geometry>
           </collision>
@@ -138,12 +138,12 @@
             <origin rpy="0 0 0" xyz="0 0 0"/>
             <geometry>
-              <mesh filename="package://trajopt_ros_examples/meshes/car_seat/visual/fence_structure.dae"/>
-            </geometry>
-            <material name="gray"/>
-          </visual>
-          <visual>
-            <origin rpy="0 0 0" xyz="0 0 0"/>
-            <geometry>
-              <mesh filename="package://trajopt_ros_examples/meshes/car_seat/visual/fence_mesh.dae"/>
+              <mesh filename="package://tesseract_ros_examples/meshes/car_seat/visual/fence_structure.dae"/>
+            </geometry>
+            <material name="gray"/>
+          </visual>
+          <visual>
+            <origin rpy="0 0 0" xyz="0 0 0"/>
+            <geometry>
+              <mesh filename="package://tesseract_ros_examples/meshes/car_seat/visual/fence_mesh.dae"/>
             </geometry>
             <material name="gray"/>
@@ -161,5 +161,5 @@
             <origin rpy="0 0 0" xyz="0 0 0"/>
             <geometry>
-              <mesh filename="package://trajopt_ros_examples/meshes/car_seat/visual/conveyor.dae"/>
+              <mesh filename="package://tesseract_ros_examples/meshes/car_seat/visual/conveyor.dae"/>
             </geometry>
             <material name="gray"/>
@@ -177,12 +177,12 @@
             <origin rpy="0 0 0" xyz="0 0 0"/>
             <geometry>
-              <mesh filename="package://trajopt_ros_examples/meshes/car_seat/visual/rail_structure.dae"/>
-            </geometry>
-            <material name="gray"/>
-          </visual>
-          <visual>
-            <origin rpy="0 0 0" xyz="0 0 0"/>
-            <geometry>
-              <mesh filename="package://trajopt_ros_examples/meshes/car_seat/visual/rail_feet.dae"/>
+              <mesh filename="package://tesseract_ros_examples/meshes/car_seat/visual/rail_structure.dae"/>
+            </geometry>
+            <material name="gray"/>
+          </visual>
+          <visual>
+            <origin rpy="0 0 0" xyz="0 0 0"/>
+            <geometry>
+              <mesh filename="package://tesseract_ros_examples/meshes/car_seat/visual/rail_feet.dae"/>
             </geometry>
             <material name="gray"/>
@@ -200,5 +200,5 @@
             <origin rpy="0 0 0" xyz="0 0 0"/>
             <geometry>
-              <mesh filename="package://trajopt_ros_examples/meshes/car_seat/visual/carriage_plate.stl"/>
+              <mesh filename="package://tesseract_ros_examples/meshes/car_seat/visual/carriage_plate.stl"/>
             </geometry>
             <material name="gray"/>
@@ -216,12 +216,12 @@
             <origin rpy="0 0 0" xyz="0 0 0"/>
             <geometry>
-              <mesh filename="package://trajopt_ros_examples/meshes/car_seat/visual/end_effector_simple.stl"/>
-            </geometry>
-            <material name="gray"/>
-          </visual>
-          <collision>
-            <origin ryp="0 0 0" xyz="0 0 0"/>
-            <geometry>
-              <mesh filename="package://trajopt_ros_examples/meshes/car_seat/visual/end_effector_simple.stl"/>
+              <mesh filename="package://tesseract_ros_examples/meshes/car_seat/visual/end_effector_simple.stl"/>
+            </geometry>
+            <material name="gray"/>
+          </visual>
+          <collision>
+            <origin ryp="0 0 0" xyz="0 0 0"/>
+            <geometry>
+              <mesh filename="package://tesseract_ros_examples/meshes/car_seat/visual/end_effector_simple.stl"/>
             </geometry>
             <material name="yellow"/>
@@ -232,75 +232,75 @@
             <origin rpy="0 0 0" xyz="0 0 0"/>
             <geometry>
-              <mesh scale="0.9 0.9 0.9" filename="package://trajopt_ros_examples/meshes/car_seat/visual/seat.dae"/>
-            </geometry>
-            <material name="gray"/>
-          </visual>
-          <collision>
-            <origin ryp="0 0 0" xyz="0 0 0"/>
-            <geometry>
-              <mesh scale="0.9 0.9 0.9" filename="package://trajopt_ros_examples/meshes/car_seat/collision/seat_1.stl"/>
-            </geometry>
-            <material name="yellow"/>
-          </collision>
-          <collision>
-            <origin ryp="0 0 0" xyz="0 0 0"/>
-            <geometry>
-              <mesh scale="0.9 0.9 0.9" filename="package://trajopt_ros_examples/meshes/car_seat/collision/seat_2.stl"/>
-            </geometry>
-            <material name="yellow"/>
-          </collision>
-          <collision>
-            <origin ryp="0 0 0" xyz="0 0 0"/>
-            <geometry>
-              <mesh scale="0.9 0.9 0.9" filename="package://trajopt_ros_examples/meshes/car_seat/collision/seat_3.stl"/>
-            </geometry>
-            <material name="yellow"/>
-          </collision>
-          <collision>
-            <origin ryp="0 0 0" xyz="0 0 0"/>
-            <geometry>
-              <mesh scale="0.9 0.9 0.9" filename="package://trajopt_ros_examples/meshes/car_seat/collision/seat_4.stl"/>
-            </geometry>
-            <material name="yellow"/>
-          </collision>
-          <collision>
-            <origin ryp="0 0 0" xyz="0 0 0"/>
-            <geometry>
-              <mesh scale="0.9 0.9 0.9" filename="package://trajopt_ros_examples/meshes/car_seat/collision/seat_5.stl"/>
-            </geometry>
-            <material name="yellow"/>
-          </collision>
-          <collision>
-            <origin ryp="0 0 0" xyz="0 0 0"/>
-            <geometry>
-              <mesh scale="0.9 0.9 0.9" filename="package://trajopt_ros_examples/meshes/car_seat/collision/seat_6.stl"/>
-            </geometry>
-            <material name="yellow"/>
-          </collision>
-          <collision>
-            <origin ryp="0 0 0" xyz="0 0 0"/>
-            <geometry>
-              <mesh scale="0.9 0.9 0.9" filename="package://trajopt_ros_examples/meshes/car_seat/collision/seat_7.stl"/>
-            </geometry>
-            <material name="yellow"/>
-          </collision>
-          <collision>
-            <origin ryp="0 0 0" xyz="0 0 0"/>
-            <geometry>
-              <mesh scale="0.9 0.9 0.9" filename="package://trajopt_ros_examples/meshes/car_seat/collision/seat_8.stl"/>
-            </geometry>
-            <material name="yellow"/>
-          </collision>
-          <collision>
-            <origin ryp="0 0 0" xyz="0 0 0"/>
-            <geometry>
-              <mesh scale="0.9 0.9 0.9" filename="package://trajopt_ros_examples/meshes/car_seat/collision/seat_9.stl"/>
-            </geometry>
-            <material name="yellow"/>
-          </collision>
-          <collision>
-            <origin ryp="0 0 0" xyz="0 0 0"/>
-            <geometry>
-              <mesh scale="0.9 0.9 0.9" filename="package://trajopt_ros_examples/meshes/car_seat/collision/seat_10.stl"/>
+              <mesh scale="0.9 0.9 0.9" filename="package://tesseract_ros_examples/meshes/car_seat/visual/seat.dae"/>
+            </geometry>
+            <material name="gray"/>
+          </visual>
+          <collision>
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
File: tesseract_ros/tesseract_examples/tesseract_examples_support/urdf/environment.xacro (robot description, xacro)
@@ -11,5 +11,5 @@
     <visual>
       <geometry>
-        <mesh filename="package://trajopt_ros_examples/meshes/pick_and_place/workcell.STL"/>
+        <mesh filename="package://tesseract_ros_examples/meshes/pick_and_place/workcell.STL"/>
       </geometry>
       <material name="light_gray"/>

File: tesseract_ros/tesseract_examples/tesseract_examples_support/urdf/grinder.xacro (robot description, xacro)
@@ -6,5 +6,5 @@
        <origin xyz="0 0 0" rpy="0 0 0" />
         <geometry>
-          <mesh filename="package://trajopt_ros_examples/meshes/puzzle_piece/grinder_visual.dae" />
+          <mesh filename="package://tesseract_ros_examples/meshes/puzzle_piece/grinder_visual.dae" />
         </geometry>
       </visual>
@@ -12,5 +12,5 @@
         <origin xyz="0 0 0" rpy="0 0 0" />
         <geometry>
-          <mesh filename="package://trajopt_ros_examples/meshes/puzzle_piece/grinder_collision.dae" />
+          <mesh filename="package://tesseract_ros_examples/meshes/puzzle_piece/grinder_collision.dae" />
         </geometry>
       </collision>
