Commit message: created a new folder for planner examples, started converting basic_cartesian_example from trajopt example to planner example

File: tesseract_ros/tesseract_examples/tesseract_examples_support/urdf/iiwa7/iiwa7.xacro (robot description, xacro)
@@ -53,5 +53,5 @@
         <origin xyz="0 0 0" rpy="0 0 0"/>
         <geometry>
-          <mesh filename="package://trajopt_ros_examples/meshes/iiwa7/visual/link_0.stl"/>
+          <mesh filename="package://tesseract_ros_examples/meshes/iiwa7/visual/link_0.stl"/>
         </geometry>
         <material name="Grey"/>
@@ -60,5 +60,5 @@
         <origin xyz="0 0 0" rpy="0 0 0"/>
         <geometry>
-          <mesh filename="package://trajopt_ros_examples/meshes/iiwa7/collision/link_0.stl"/>
+          <mesh filename="package://tesseract_ros_examples/meshes/iiwa7/collision/link_0.stl"/>
         </geometry>
         <material name="Grey"/>
@@ -94,5 +94,5 @@
         <origin xyz="0 0 0.0075" rpy="0 0 0"/>
         <geometry>
-          <mesh filename="package://trajopt_ros_examples/meshes/iiwa7/visual/link_1.stl"/>
+          <mesh filename="package://tesseract_ros_examples/meshes/iiwa7/visual/link_1.stl"/>
         </geometry>
         <material name="Orange"/>
@@ -101,5 +101,5 @@
         <origin xyz="0 0 0.0075" rpy="0 0 0"/>
         <geometry>
-          <mesh filename="package://trajopt_ros_examples/meshes/iiwa7/collision/link_1.stl"/>
+          <mesh filename="package://tesseract_ros_examples/meshes/iiwa7/collision/link_1.stl"/>
         </geometry>
         <material name="Orange"/>
@@ -128,12 +128,12 @@
         <origin xyz="0 0 0" rpy="0 0 0"/>
         <geometry>
-          <mesh filename="package://trajopt_ros_examples/meshes/iiwa7/visual/link_2.stl"/>
-        </geometry>
-        <material name="Orange"/>
-      </visual>
-      <collision>
-        <origin xyz="0 0 0" rpy="0 0 0"/>
-        <geometry>
-          <mesh filename="package://trajopt_ros_examples/meshes/iiwa7/collision/link_2.stl"/>
+          <mesh filename="package://tesseract_ros_examples/meshes/iiwa7/visual/link_2.stl"/>
+        </geometry>
+        <material name="Orange"/>
+      </visual>
+      <collision>
+        <origin xyz="0 0 0" rpy="0 0 0"/>
+        <geometry>
+          <mesh filename="package://tesseract_ros_examples/meshes/iiwa7/collision/link_2.stl"/>
         </geometry>
         <material name="Orange"/>
@@ -162,5 +162,5 @@
         <origin xyz="0 0 -0.026" rpy="0 0 0"/>
         <geometry>
-          <mesh filename="package://trajopt_ros_examples/meshes/iiwa7/visual/link_3.stl"/>
+          <mesh filename="package://tesseract_ros_examples/meshes/iiwa7/visual/link_3.stl"/>
         </geometry>
         <material name="Orange"/>
@@ -169,5 +169,5 @@
         <origin xyz="0 0 -0.026" rpy="0 0 0"/>
         <geometry>
-          <mesh filename="package://trajopt_ros_examples/meshes/iiwa7/collision/link_3.stl"/>
+          <mesh filename="package://tesseract_ros_examples/meshes/iiwa7/collision/link_3.stl"/>
         </geometry>
         <material name="Orange"/>
@@ -196,12 +196,12 @@
         <origin xyz="0 0 0" rpy="0 0 0"/>
         <geometry>
-          <mesh filename="package://trajopt_ros_examples/meshes/iiwa7/visual/link_4.stl"/>
-        </geometry>
-        <material name="Orange"/>
-      </visual>
-      <collision>
-        <origin xyz="0 0 0" rpy="0 0 0"/>
-        <geometry>
-          <mesh filename="package://trajopt_ros_examples/meshes/iiwa7/collision/link_4.stl"/>
+          <mesh filename="package://tesseract_ros_examples/meshes/iiwa7/visual/link_4.stl"/>
+        </geometry>
+        <material name="Orange"/>
+      </visual>
+      <collision>
+        <origin xyz="0 0 0" rpy="0 0 0"/>
+        <geometry>
+          <mesh filename="package://tesseract_ros_examples/meshes/iiwa7/collision/link_4.stl"/>
         </geometry>
         <material name="Orange"/>
@@ -230,5 +230,5 @@
         <origin xyz="0 0 -0.026" rpy="0 0 0"/>
         <geometry>
-          <mesh filename="package://trajopt_ros_examples/meshes/iiwa7/visual/link_5.stl"/>
+          <mesh filename="package://tesseract_ros_examples/meshes/iiwa7/visual/link_5.stl"/>
         </geometry>
         <material name="Orange"/>
@@ -237,5 +237,5 @@
         <origin xyz="0 0 -0.026" rpy="0 0 0"/>
         <geometry>
-          <mesh filename="package://trajopt_ros_examples/meshes/iiwa7/collision/link_5.stl"/>
+          <mesh filename="package://tesseract_ros_examples/meshes/iiwa7/collision/link_5.stl"/>
         </geometry>
         <material name="Orange"/>
@@ -264,12 +264,12 @@
         <origin xyz="0 0 0" rpy="0 0 0"/>
         <geometry>
-          <mesh filename="package://trajopt_ros_examples/meshes/iiwa7/visual/link_6.stl"/>
-        </geometry>
-        <material name="Orange"/>
-      </visual>
-      <collision>
-        <origin xyz="0 0 0" rpy="0 0 0"/>
-        <geometry>
-          <mesh filename="package://trajopt_ros_examples/meshes/iiwa7/collision/link_6.stl"/>
+          <mesh filename="package://tesseract_ros_examples/meshes/iiwa7/visual/link_6.stl"/>
+        </geometry>
+        <material name="Orange"/>
+      </visual>
+      <collision>
+        <origin xyz="0 0 0" rpy="0 0 0"/>
+        <geometry>
+          <mesh filename="package://tesseract_ros_examples/meshes/iiwa7/collision/link_6.stl"/>
         </geometry>
         <material name="Orange"/>
@@ -298,5 +298,5 @@
         <origin xyz="0 0 -0.0005" rpy="0 0 0"/>
         <geometry>
-          <mesh filename="package://trajopt_ros_examples/meshes/iiwa7/visual/link_7.stl"/>
+          <mesh filename="package://tesseract_ros_examples/meshes/iiwa7/visual/link_7.stl"/>
         </geometry>
         <material name="Grey"/>
@@ -305,5 +305,5 @@
         <origin xyz="0 0 -0.0005" rpy="0 0 0"/>
         <geometry>
-          <mesh filename="package://trajopt_ros_examples/meshes/iiwa7/collision/link_7.stl"/>
+          <mesh filename="package://tesseract_ros_examples/meshes/iiwa7/collision/link_7.stl"/>
         </geometry>
         <material name="Grey"/>

File: tesseract_ros/tesseract_examples/tesseract_examples_support/urdf/lbr_iiwa_14_r820_macro.xacro (robot description, xacro)
@@ -7,5 +7,5 @@
         <origin xyz="0 0 0" rpy="0 0 0" />
         <geometry>
-          <mesh filename="package://trajopt_ros_examples/meshes/lbr_iiwa_14_r820/visual/base_link.dae" />
+          <mesh filename="package://tesseract_examples_support/meshes/lbr_iiwa_14_r820/visual/base_link.dae" />
         </geometry>
       </visual>
@@ -13,5 +13,5 @@
         <origin xyz="0 0 0" rpy="0 0 0" />
         <geometry>
-          <mesh filename="package://trajopt_ros_examples/meshes/lbr_iiwa_14_r820/collision/base_link.stl" />
+          <mesh filename="package://tesseract_examples_support/meshes/lbr_iiwa_14_r820/collision/base_link.stl" />
         </geometry>
       </collision>
@@ -21,5 +21,5 @@
         <origin xyz="0 0 0" rpy="0 0 0" />
         <geometry>
-          <mesh filename="package://trajopt_ros_examples/meshes/lbr_iiwa_14_r820/visual/link_1.dae" />
+          <mesh filename="package://tesseract_examples_support/meshes/lbr_iiwa_14_r820/visual/link_1.dae" />
         </geometry>
       </visual>
@@ -27,5 +27,5 @@
         <origin xyz="0 0 0" rpy="0 0 0" />
         <geometry>
-          <mesh filename="package://trajopt_ros_examples/meshes/lbr_iiwa_14_r820/collision/link_1.stl" />
+          <mesh filename="package://tesseract_examples_support/meshes/lbr_iiwa_14_r820/collision/link_1.stl" />
         </geometry>
       </collision>
@@ -35,5 +35,5 @@
         <origin xyz="0 0 0" rpy="0 0 0" />
         <geometry>
-          <mesh filename="package://trajopt_ros_examples/meshes/lbr_iiwa_14_r820/visual/link_2.dae" />
+          <mesh filename="package://tesseract_examples_support/meshes/lbr_iiwa_14_r820/visual/link_2.dae" />
         </geometry>
       </visual>
@@ -41,5 +41,5 @@
         <origin xyz="0 0 0" rpy="0 0 0" />
         <geometry>
-          <mesh filename="package://trajopt_ros_examples/meshes/lbr_iiwa_14_r820/collision/link_2.stl" />
+          <mesh filename="package://tesseract_examples_support/meshes/lbr_iiwa_14_r820/collision/link_2.stl" />
         </geometry>
       </collision>
@@ -49,5 +49,5 @@
         <origin xyz="0 0 0" rpy="0 0 0" />
         <geometry>
-          <mesh filename="package://trajopt_ros_examples/meshes/lbr_iiwa_14_r820/visual/link_3.dae" />
+          <mesh filename="package://tesseract_examples_support/meshes/lbr_iiwa_14_r820/visual/link_3.dae" />
         </geometry>
       </visual>
@@ -55,5 +55,5 @@
         <origin xyz="0 0 0" rpy="0 0 0" />
         <geometry>
-          <mesh filename="package://trajopt_ros_examples/meshes/lbr_iiwa_14_r820/collision/link_3.stl" />
+          <mesh filename="package://tesseract_examples_support/meshes/lbr_iiwa_14_r820/collision/link_3.stl" />
         </geometry>
       </collision>
@@ -63,5 +63,5 @@
         <origin xyz="0 0 0" rpy="0 0 0" />
         <geometry>
-          <mesh filename="package://trajopt_ros_examples/meshes/lbr_iiwa_14_r820/visual/link_4.dae" />
+          <mesh filename="package://tesseract_examples_support/meshes/lbr_iiwa_14_r820/visual/link_4.dae" />
         </geometry>
       </visual>
@@ -69,5 +69,5 @@
         <origin xyz="0 0 0" rpy="0 0 0" />
         <geometry>
-          <mesh filename="package://trajopt_ros_examples/meshes/lbr_iiwa_14_r820/collision/link_4.stl" />
+          <mesh filename="package://tesseract_examples_support/meshes/lbr_iiwa_14_r820/collision/link_4.stl" />
         </geometry>
       </collision>
@@ -77,5 +77,5 @@
         <origin xyz="0 0 0" rpy="0 0 0" />
         <geometry>
-          <mesh filename="package://trajopt_ros_examples/meshes/lbr_iiwa_14_r820/visual/link_5.dae" />
+          <mesh filename="package://tesseract_examples_support/meshes/lbr_iiwa_14_r820/visual/link_5.dae" />
         </geometry>
       </visual>
@@ -83,5 +83,5 @@
         <origin xyz="0 0 0" rpy="0 0 0" />
         <geometry>
-          <mesh filename="package://trajopt_ros_examples/meshes/lbr_iiwa_14_r820/collision/link_5.stl" />
+          <mesh filename="package://tesseract_examples_support/meshes/lbr_iiwa_14_r820/collision/link_5.stl" />
         </geometry>
       </collision>
@@ -91,5 +91,5 @@
         <origin xyz="0 0 0" rpy="0 0 0" />
         <geometry>
-          <mesh filename="package://trajopt_ros_examples/meshes/lbr_iiwa_14_r820/visual/link_6.dae" />
+          <mesh filename="package://tesseract_examples_support/meshes/lbr_iiwa_14_r820/visual/link_6.dae" />
         </geometry>
       </visual>
@@ -97,5 +97,5 @@
         <origin xyz="0 0 0" rpy="0 0 0" />
         <geometry>
-          <mesh filename="package://trajopt_ros_examples/meshes/lbr_iiwa_14_r820/collision/link_6.stl" />
+          <mesh filename="package://tesseract_examples_support/meshes/lbr_iiwa_14_r820/collision/link_6.stl" />
         </geometry>
       </collision>
@@ -105,5 +105,5 @@
         <origin xyz="0 0 0" rpy="0 0 0" />
         <geometry>
-          <mesh filename="package://trajopt_ros_examples/meshes/lbr_iiwa_14_r820/visual/link_7.dae" />
+          <mesh filename="package://tesseract_examples_support/meshes/lbr_iiwa_14_r820/visual/link_7.dae" />
         </geometry>
       </visual>
@@ -111,5 +111,5 @@
         <origin xyz="0 0 0" rpy="0 0 0" />
         <geometry>
-          <mesh filename="package://trajopt_ros_examples/meshes/lbr_iiwa_14_r820/collision/link_7.stl" />
+          <mesh filename="package://tesseract_examples_support/meshes/lbr_iiwa_14_r820/collision/link_7.stl" />
         </geometry>
       </collision>

File: tesseract_ros/tesseract_examples/tesseract_examples_support/urdf/puzzle_mount.xacro (robot description, xacro)
@@ -7,10 +7,10 @@
       <visual>
         <geometry>
-          <mesh filename="package://trajopt_ros_examples/meshes/puzzle_piece/puzzle_mount.stl" />
+          <mesh filename="package://tesseract_ros_examples/meshes/puzzle_piece/puzzle_mount.stl" />
         </geometry>>
       </visual>
       <collision>
         <geometry>
-          <mesh filename="package://trajopt_ros_examples/meshes/puzzle_piece/puzzle_mount.stl" />
+          <mesh filename="package://tesseract_ros_examples/meshes/puzzle_piece/puzzle_mount.stl" />
         </geometry>
       </collision>
@@ -31,10 +31,10 @@
       <visual>
         <geometry>
-          <mesh filename="package://trajopt_ros_examples/meshes/puzzle_piece/puzzle_bent.dae" />
+          <mesh filename="package://tesseract_ros_examples/meshes/puzzle_piece/puzzle_bent.dae" />
         </geometry>
       </visual>
       <collision>
         <geometry>
-          <mesh filename="package://trajopt_ros_examples/meshes/puzzle_piece/puzzle_bent.dae" />
+          <mesh filename="package://tesseract_ros_examples/meshes/puzzle_piece/puzzle_bent.dae" />
         </geometry>
       </collision>

File: tesseract_ros/tesseract_examples/tesseract_examples_support/urdf/sia20d_macro.xacro (robot description, xacro)
@@ -6,5 +6,5 @@
 			<visual>
 				<geometry>
-                                        <mesh filename="package://trajopt_ros_examples/meshes/sia20d/visual/MOTOMAN_BASE.stl" />
+                                        <mesh filename="package://tesseract_ros_examples/meshes/sia20d/visual/MOTOMAN_BASE.stl" />
 				</geometry>
 				<material name="blue">
@@ -14,5 +14,5 @@
 			<collision>
 				<geometry>
-                                        <mesh filename="package://trajopt_ros_examples/meshes/sia20d/collision/MOTOMAN_BASE.stl" />
+                                        <mesh filename="package://tesseract_ros_examples/meshes/sia20d/collision/MOTOMAN_BASE.stl" />
 				</geometry>
 				<material name="yellow">
@@ -25,5 +25,5 @@
 				<origin rpy="0 0 3.1416" xyz="0 0 0"/>
 				<geometry>
-                                        <mesh filename="package://trajopt_ros_examples/meshes/sia20d/visual/MOTOMAN_AXIS_S.stl"/>
+                                        <mesh filename="package://tesseract_ros_examples/meshes/sia20d/visual/MOTOMAN_AXIS_S.stl"/>
 				</geometry>
 				<material name="silver">
@@ -34,5 +34,5 @@
 				<origin rpy="0 0 3.1416" xyz="0 0 0"/>
 				<geometry>
-                                        <mesh filename="package://trajopt_ros_examples/meshes/sia20d/collision/MOTOMAN_AXIS_S.stl" />
+                                        <mesh filename="package://tesseract_ros_examples/meshes/sia20d/collision/MOTOMAN_AXIS_S.stl" />
 				</geometry>
 				<material name="yellow"/>
@@ -43,5 +43,5 @@
 				<origin rpy="1.57 3.1416 3.1416" xyz="0 0 0"/>
 				<geometry>
-                                        <mesh filename="package://trajopt_ros_examples/meshes/sia20d/visual/MOTOMAN_AXIS_L.stl"/>
+                                        <mesh filename="package://tesseract_ros_examples/meshes/sia20d/visual/MOTOMAN_AXIS_L.stl"/>
 				</geometry>
 				<material name="blue"/>
@@ -50,5 +50,5 @@
 				<origin rpy="1.57 3.1416 3.1416" xyz="0 0 0"/>
 				<geometry>
-                                        <mesh filename="package://trajopt_ros_examples/meshes/sia20d/collision/MOTOMAN_AXIS_L.stl"/>
+                                        <mesh filename="package://tesseract_ros_examples/meshes/sia20d/collision/MOTOMAN_AXIS_L.stl"/>
 				</geometry>
 				<material name="yellow"/>
@@ -59,5 +59,5 @@
 				<origin rpy="0 0 0" xyz="0 0 0"/>
 				<geometry>
-                                        <mesh filename="package://trajopt_ros_examples/meshes/sia20d/visual/MOTOMAN_AXIS_E.stl"/>
+                                        <mesh filename="package://tesseract_ros_examples/meshes/sia20d/visual/MOTOMAN_AXIS_E.stl"/>
 				</geometry>
 				<material name="silver"/>
@@ -66,5 +66,5 @@
 				<origin rpy="0 0 0" xyz="0 0 0"/>
 				<geometry>
-                                        <mesh filename="package://trajopt_ros_examples/meshes/sia20d/collision/MOTOMAN_AXIS_E.stl"/>
+                                        <mesh filename="package://tesseract_ros_examples/meshes/sia20d/collision/MOTOMAN_AXIS_E.stl"/>
 				</geometry>
 				<material name="yellow"/>
@@ -75,5 +75,5 @@
 				<origin rpy="1.57 -3.1415 3.1416" xyz="0 0 0"/>
 				<geometry>
-                                        <mesh filename="package://trajopt_ros_examples/meshes/sia20d/visual/MOTOMAN_AXIS_U.stl"/>
+                                        <mesh filename="package://tesseract_ros_examples/meshes/sia20d/visual/MOTOMAN_AXIS_U.stl"/>
 				</geometry>
 				<material name="blue"/>
@@ -82,5 +82,5 @@
 				<origin rpy="1.57 -3.1415 3.1416" xyz="0 0 0"/>
 				<geometry>
-                                        <mesh filename="package://trajopt_ros_examples/meshes/sia20d/collision/MOTOMAN_AXIS_U.stl"/>
+                                        <mesh filename="package://tesseract_ros_examples/meshes/sia20d/collision/MOTOMAN_AXIS_U.stl"/>
 				</geometry>
 				<material name="yellow"/>
@@ -91,5 +91,5 @@
 				<origin rpy="0 0 0" xyz="0 0 0"/>
 				<geometry>
-                                        <mesh filename="package://trajopt_ros_examples/meshes/sia20d/visual/MOTOMAN_AXIS_R.stl"/>
+                                        <mesh filename="package://tesseract_ros_examples/meshes/sia20d/visual/MOTOMAN_AXIS_R.stl"/>
 				</geometry>
 				<material name="silver"/>
@@ -98,5 +98,5 @@
 				<origin rpy="0 0 0" xyz="0 0 0"/>
 				<geometry>
-                                        <mesh filename="package://trajopt_ros_examples/meshes/sia20d/collision/MOTOMAN_AXIS_R.stl"/>
+                                        <mesh filename="package://tesseract_ros_examples/meshes/sia20d/collision/MOTOMAN_AXIS_R.stl"/>
 				</geometry>
 				<material name="yellow"/>
@@ -107,5 +107,5 @@
 				<origin rpy="-1.57 0 0" xyz="0 0 0"/>
 				<geometry>
-                                        <mesh filename="package://trajopt_ros_examples/meshes/sia20d/visual/MOTOMAN_AXIS_B.stl"/>
+                                        <mesh filename="package://tesseract_ros_examples/meshes/sia20d/visual/MOTOMAN_AXIS_B.stl"/>
 				</geometry>
 				<material name="blue"/>
@@ -114,5 +114,5 @@
 				<origin rpy="-1.57 0 0" xyz="0 0 0"/>
 				<geometry>
-                                        <mesh filename="package://trajopt_ros_examples/meshes/sia20d/collision/MOTOMAN_AXIS_B.stl"/>
+                                        <mesh filename="package://tesseract_ros_examples/meshes/sia20d/collision/MOTOMAN_AXIS_B.stl"/>
 				</geometry>
 				<material name="yellow"/>
@@ -122,5 +122,5 @@
 			<visual>
 				<geometry>
-                                        <mesh filename="package://trajopt_ros_examples/meshes/sia20d/visual/MOTOMAN_AXIS_T.stl" />
+                                        <mesh filename="package://tesseract_ros_examples/meshes/sia20d/visual/MOTOMAN_AXIS_T.stl" />
 				</geometry>
 				<material name="silver"/>
@@ -128,5 +128,5 @@
 			<collision>
 				<geometry>
-                                        <mesh filename="package://trajopt_ros_examples/meshes/sia20d/collision/MOTOMAN_AXIS_T.stl" />
+                                        <mesh filename="package://tesseract_ros_examples/meshes/sia20d/collision/MOTOMAN_AXIS_T.stl" />
 				</geometry>
 				<material name="yellow"/>
